Commit message: Update urdf

File: urdf/raspicat.urdf.xacro (robot description, xacro)
@@ -16,5 +16,5 @@
   <xacro:arg name="lidar_frame"           default="lidar_link"/>
   <!-- =============== Xacro property =============== -->
-  <xacro:property name="lidar_mount_z" value="0.0"/>
+  <xacro:property name="lidar_mount_z" value="0.18"/>
   <xacro:property name="lidar_sensor_z" value="0.055"/>
   <!-- =============== Xacro include =============== -->
@@ -53,5 +53,5 @@
   <!-- Sensors -->
   <xacro:lidar_mount prefix="lidar_mount" parent="base_link">
-    <origin xyz="0.144 0 ${lidar_mount_z - 0.0262}" rpy="0 0 0"/>
+    <origin xyz="-0.144 0 ${lidar_mount_z - 0.0262}" rpy="0 0 0"/>
   </xacro:lidar_mount>
   <xacro:lidar_sensor prefix="laser" parent="lidar_mount_link" lidar_frame="$(arg lidar_frame)">

Commit message: Feature GNSS

File: urdf/raspicat.urdf.xacro (robot description, xacro)
@@ -8,4 +8,5 @@
   <xacro:arg name="camera_gazebo_plugin"  default="true"/>
   <xacro:arg name="imu_gazebo_plugin"     default="true"/>
+  <xacro:arg name="gnss_gazebo_plugin"    default="true"/>
   <xacro:arg name="diffdrive_pub_tf"      default="true"/>
   <xacro:arg name="jointstate"            default="true"/>
@@ -27,4 +28,5 @@
   <xacro:include filename="$(find raspicat_description)/urdf/sensors/realsense_d435.urdf.xacro"/>
   <xacro:include filename="$(find raspicat_description)/urdf/sensors/imu.urdf.xacro"/>
+  <xacro:include filename="$(find raspicat_description)/urdf/sensors/gnss.urdf.xacro"/>
   <!-- =============== Link & Joint =============== -->
   <link name="base_footprint"/>
@@ -78,4 +80,8 @@
     <origin xyz="0 0 0.14" rpy="${M_PI} 0 0"/>
   </xacro:imu_sensor>
+  <!-- Gnss -->
+  <xacro:gnss_sensor prefix="gnss" parent="base_link">
+    <origin xyz="0 0 0.14" rpy="0 0 0"/>
+  </xacro:gnss_sensor>
   <!-- =============== Gazebo =============== -->
   <xacro:if value="$(arg gazebo_plugin)">
@@ -113,4 +119,12 @@
         prefix="imu" parent="base_link"/>
     </xacro:if>
+    <!-- Gnss -->
+    <xacro:if value="$(arg gnss_gazebo_plugin)">
+      <spherical_coordinates>
+        <heading_deg>180</heading_deg>
+      </spherical_coordinates>
+      <xacro:gnss_sensor_gazebo
+        prefix="gnss" parent="base_link"/>
+    </xacro:if>
   </xacro:if>
 </robot>

Commit message: Add/secondLiDAR

File: urdf/raspicat.urdf.xacro (robot description, xacro)
@@ -58,4 +58,13 @@
     <origin xyz="0 0 ${lidar_sensor_z}" rpy="0 0 0"/>
   </xacro:lidar_sensor>
+    <!-- Add/LiDAR2 -->
+  <xacro:lidar_mount prefix="lidar2_mount" parent="base_link">
+    <origin xyz="-0.2425 0 0.706" rpy="0 0.29655556 0"/>
+      <!-- 地面から取付台: 0.665m,取付台からマウント（真ん中）: 0.041m,マウントの取り付け角度: 17度 -->
+  </xacro:lidar_mount>
+  <xacro:lidar2_sensor prefix="laser2" parent="lidar2_mount_link" lidar_frame="lidar2_link">
+    <origin xyz="0 0 ${lidar_sensor_z}" rpy="0 0 0"/>
+  </xacro:lidar2_sensor>
+  <!--  -->
   <xacro:ultrasonic_sensor prefix="right_side" parent="base_link">
     <origin xyz="0.1055 -0.1165 -0.00795" rpy="0 0 -0.837758"/>

File: urdf/sensors/lidar.urdf.xacro (robot description, xacro)
@@ -18,3 +18,11 @@
     <link name="${lidar_frame}"/>
   </xacro:macro>
+  <xacro:macro name="lidar2_sensor" params="prefix parent lidar_frame *joint_origin">
+    <joint name="lidar2_frame_joint" type="fixed">
+      <xacro:insert_block name="joint_origin"/>
+      <parent link="${parent}"/>
+      <child link="lidar2_link"/>
+    </joint>
+    <link name="lidar2_link"/>
+  </xacro:macro>
 </robot>

Commit message: Fix/axisCoordinate of lidar2

File: urdf/raspicat.urdf.xacro (robot description, xacro)
@@ -60,5 +60,5 @@
     <!-- Add/LiDAR2 -->
   <xacro:lidar_mount prefix="lidar2_mount" parent="base_link">
-    <origin xyz="-0.2425 0 0.706" rpy="0 0.29655556 0"/>
+    <origin xyz="-0.155 0 0.706" rpy="0 0.29655556 0"/>
       <!-- 地面から取付台: 0.665m,取付台からマウント（真ん中）: 0.041m,マウントの取り付け角度: 17度 -->
   </xacro:lidar_mount>

Commit message: Update/axiscoordinate of lidar2

File: urdf/raspicat.urdf.xacro (robot description, xacro)
@@ -60,5 +60,5 @@
     <!-- Add/LiDAR2 -->
   <xacro:lidar_mount prefix="lidar2_mount" parent="base_link">
-    <origin xyz="-0.155 0 0.706" rpy="0 0.29655556 0"/>
+    <origin xyz="-0.240 0 0.706" rpy="0 0.29655556 0"/>
       <!-- 地面から取付台: 0.665m,取付台からマウント（真ん中）: 0.041m,マウントの取り付け角度: 17度 -->
   </xacro:lidar_mount>

Commit message: Update/axiscoordinate of lidar2

File: urdf/raspicat.urdf.xacro (robot description, xacro)
@@ -16,5 +16,5 @@
   <xacro:arg name="lidar_frame"           default="lidar_link"/>
   <!-- =============== Xacro property =============== -->
-  <xacro:property name="lidar_mount_z" value="0.0"/>
+  <xacro:property name="lidar_mount_z" value="0.23"/>
   <xacro:property name="lidar_sensor_z" value="0.055"/>
   <!-- =============== Xacro include =============== -->
@@ -53,5 +53,5 @@
   <!-- Sensors -->
   <xacro:lidar_mount prefix="lidar_mount" parent="base_link">
-    <origin xyz="0.144 0 ${lidar_mount_z - 0.0262}" rpy="0 0 0"/>
+    <origin xyz="0.06 0 ${lidar_mount_z - 0.0262}" rpy="0 0 0"/>
   </xacro:lidar_mount>
   <xacro:lidar_sensor prefix="laser" parent="lidar_mount_link" lidar_frame="$(arg lidar_frame)">

Commit message: Update positional relationship

File: urdf/raspicat.urdf.xacro (robot description, xacro)
@@ -55,8 +55,10 @@
   <!-- Sensors -->
   <xacro:lidar_mount prefix="lidar_mount" parent="base_footprint">
-    <origin xyz="-0.355 0 0.335" rpy="0 0 0"/>
+	  <!--<origin xyz="-0.355 0 0.335" rpy="0 0 0"/>-->
+    <origin xyz="-0.3 0 0.285" rpy="0 0 0"/>
   </xacro:lidar_mount>
   <xacro:lidar_sensor prefix="laser" parent="lidar_mount_link" lidar_frame="$(arg lidar_frame)">
-    <origin xyz="0 0 0.045" rpy="0 0.1222 0"/>
+	  <!-- <origin xyz="0 0 0.045" rpy="0 0.1222 0"/>-->
+    <origin xyz="0 0 0.045" rpy="0 0 0"/>
   </xacro:lidar_sensor>
   <!-- ultrasonic_sensor
@@ -78,10 +80,12 @@
   </xacro:realsensed435_sensor> -->
   <!-- Imu -->
-  <xacro:imu_sensor prefix="imu" parent="base_footprint">
-    <origin xyz="-0.355 0 0.38" rpy="0 0.1222 0"/>
+  <xacro:imu_sensor prefix="imu" parent="lidar_mount_link">
+	  <!--<origin xyz="-0.355 0 0.38" rpy="0 0.1222 0"/>-->
+    <origin xyz="-0 0 0" rpy="0 0 0"/>
   </xacro:imu_sensor>
   <!-- Gnss -->
   <xacro:gnss_sensor prefix="gnss" parent="base_footprint">
-    <origin xyz="-0.22 0 0.3" rpy="0 0 0"/>
+	  <!--<origin xyz="-0.22 0 0.3" rpy="0 0 0"/>-->
+    <origin xyz="-0.34 0 0.585" rpy="0 0 0"/>
   </xacro:gnss_sensor>
   <!-- =============== Gazebo =============== -->

Commit message: Change imu pose

File: urdf/raspicat.urdf.xacro (robot description, xacro)
@@ -80,7 +80,8 @@
   </xacro:realsensed435_sensor> -->
   <!-- Imu -->
-  <xacro:imu_sensor prefix="imu" parent="lidar_mount_link">
+	  <!--<xacro:imu_sensor prefix="imu" parent="lidar_mount_link">-->
+  <xacro:imu_sensor prefix="imu" parent="base_link">
 	  <!--<origin xyz="-0.355 0 0.38" rpy="0 0.1222 0"/>-->
-    <origin xyz="-0 0 0" rpy="0 0 0"/>
+    <origin xyz="-0 0 0" rpy="3.14 0 0"/>
   </xacro:imu_sensor>
   <!-- Gnss -->

Commit message: Change IMU pose

File: urdf/raspicat.urdf.xacro (robot description, xacro)
@@ -83,5 +83,5 @@
   <xacro:imu_sensor prefix="imu" parent="base_link">
 	  <!--<origin xyz="-0.355 0 0.38" rpy="0 0.1222 0"/>-->
-    <origin xyz="-0 0 0" rpy="3.14 0 0"/>
+    <origin xyz="0 0 0" rpy="0 0 0"/>
   </xacro:imu_sensor>
   <!-- Gnss -->

Commit message: Change lidar position

File: urdf/raspicat.urdf.xacro (robot description, xacro)
@@ -56,5 +56,5 @@
   <xacro:lidar_mount prefix="lidar_mount" parent="base_footprint">
 	  <!--<origin xyz="-0.355 0 0.335" rpy="0 0 0"/>-->
-    <origin xyz="-0.3 0 0.285" rpy="0 0 0"/>
+    <origin xyz="0.055 0 0.235" rpy="0 0 0"/>
   </xacro:lidar_mount>
   <xacro:lidar_sensor prefix="laser" parent="lidar_mount_link" lidar_frame="$(arg lidar_frame)">
